File: Hardware/Radio clock rebuild.kicad_sch (KiCad schematic)
At the start: 6 parts, among them U1 ATmega328P-P, U2 ES100_module-DIP, U3 LP2950-3.3_TO92, U4 DS1307+, U5 LM7805_TO220

Commit message: starting to flush out the hardware
Parts:
- added BT1: CR1220, symbol Device:Battery_Cell
- added Q1, Q2, Q3: 2N7000, Package_TO_SOT_THT:TO-92_Inline, symbol Transistor_FET:2N7000
- added R1, R2, R3: 10K, symbol Device:R
- added R4: 1K, symbol Device:R
- added R5: 2K2, symbol Device:R
- added Y1: 32768Hz, 12.5pF, symbol Device:Crystal_Small
Connections:
- net +5V: now also U4.8 (VCC), R1.1, R2.1, R3.1
- net GND: now also U2.1 (GND), U4.4 (GND), BT1.2 (-), R5.2
- net D13: now reaches U1.13 (PD7)
- net D13: now also R4.1
- net SDA: now reaches U1.27 (PC4)
- net SDA: now also U4.5 (SDA), Q3.3 (D), R3.2
- net SCL: now reaches U1.28 (PC5)
- net SCL: now also U4.6 (SCL), Q2.3 (D), R2.2
- net D2: now reaches U1.4 (PD2)
- net D2: now also Q1.3 (D), R1.2
- net at U2.2 (EN): now also R4.2, R5.1
- net at U2.3 (SDA): now also Q3.1 (S)
- net at U2.4 (SCL): now also Q2.1 (S)
- net at U2.5 (IRQ): now also Q1.1 (S)
- net +3.3V: now reaches U2.6 (3.3v)
- net +3.3V: now also Q1.2 (G), Q2.2 (G), Q3.2 (G)
- net at U4.1 (X1): now also Y1.2
- net at U4.2 (X2): now also Y1.1
- net at U4.3 (VBAT): now also BT1.1 (+)
- no-connect marks 1 -> 2
Other:
- note added: "ES100 Module"
- note added: "ES100 is a 3.3 volt only device."
- note added: "RTC DS1307"
- moved on the sheet: DS1, U2, U4
